File: Hardware/CarTablet.kicad_pcb (KiCad board)
At the start: 2 copper layers, 100 x 70 mm, 156 parts, among them IC1 TPS54540B-Q1, IC2 NCP81239, IC3 EZ-PD_CCG2, J1 ENABLE_KL15, J11 PD_to_USB_Hub, J12 USB_Tablet_Input, J13 USB_Hub_Output, J14 JTAG, J2 Anschluss, J4 ISP, J8 Arduino, K1 IM23GR, Q1 NTTFS4C13NTAG, Q2 NTTFS4C13NTAG, Q3 NTTFS4C13NTAG, Q4 NTTFS4C13NTAG, Q5 NTTFS4C13NTAG, Q6 FDG6335N, T1 MUN5313DW, U1 TJA1042T, U2 MCP2515-xSO, U3 ATmega328P-AU, U4 FT232RL, Y1 16 MHz, Y2 8 MHz

Commit message: V1.0 as ordered at JLCPCB
Parts:
- added C56: 10nF, Capacitor_SMD:C_0805_2012Metric_Pad1.15x1.40mm_HandSolder, F.Cu at (56.1, 106.3)
- added C57: 10nF, Capacitor_SMD:C_0805_2012Metric_Pad1.15x1.40mm_HandSolder, F.Cu at (71.4, 100.9)
- added D12: 100V, Diode_SMD:D_SMB_Handsoldering, F.Cu at (56.4, 100.6)
- added D13: 100V, Diode_SMD:D_SMB_Handsoldering, F.Cu at (71.7, 95.3)
- added D14: 4.7V, Diode_SMD:D_SMB_Handsoldering, F.Cu at (64.5, 102.4)
- added D15: 4.7V, Diode_SMD:D_SMB_Handsoldering, F.Cu at (71.7, 104.4)
- added D16: BZX84B33, Package_TO_SOT_SMD:SOT-23, F.Cu at (84.4, 94.9)
- added D17: BZX84B33, Package_TO_SOT_SMD:SOT-23, F.Cu at (97.0, 93.4)
- added G***: LOGO, Logo2:370z, F.Cu at (67.5, 123.3)
- added J3: I/O Expander, Hella_Bauteile:Molex_0901303208, F.Cu at (63.1, 114.5)
- added R55: 10k, Resistor_SMD:R_0805_2012Metric_Pad1.15x1.40mm_HandSolder, F.Cu at (56.1, 104.1)
- added R56: 10k, Resistor_SMD:R_0805_2012Metric_Pad1.15x1.40mm_HandSolder, F.Cu at (71.4, 98.8)
- added R57: 10k, Resistor_SMD:R_0805_2012Metric_Pad1.15x1.40mm_HandSolder, F.Cu at (59.1, 105.3)
- added R58: 10k, Resistor_SMD:R_0805_2012Metric_Pad1.15x1.40mm_HandSolder, F.Cu at (74.4, 99.8)
- added R59: 1k, Resistor_SMD:R_0805_2012Metric_Pad1.15x1.40mm_HandSolder, F.Cu at (61.2, 105.3)
- added R60: 1k, Resistor_SMD:R_0805_2012Metric_Pad1.15x1.40mm_HandSolder, F.Cu at (76.5, 99.8)
- added R61: 10k, Resistor_SMD:R_0805_2012Metric_Pad1.15x1.40mm_HandSolder, F.Cu at (91.3, 95.5)
- added R62: 150, Resistor_SMD:R_0805_2012Metric_Pad1.15x1.40mm_HandSolder, F.Cu at (91.3, 93.4)
- added R63: 10k, Resistor_SMD:R_0805_2012Metric_Pad1.15x1.40mm_HandSolder, F.Cu at (103.8, 94.1)
- added R64: 150, Resistor_SMD:R_0805_2012Metric_Pad1.15x1.40mm_HandSolder, F.Cu at (103.8, 92.0)
- added REF**: Stitching_Via_0.6mm, Hella_Bauteile:Stitching_Via_0.6mm, F.Cu at (100.3, 116.1)
- added REF**: Stitching_Via_0.6mm, Hella_Bauteile:Stitching_Via_0.6mm, F.Cu at (99.1, 117.3)
- added REF**: Stitching_Via_0.6mm, Hella_Bauteile:Stitching_Via_0.6mm, F.Cu at (100.3, 118.6)
- added REF**: Stitching_Via_0.6mm, Hella_Bauteile:Stitching_Via_0.6mm, F.Cu at (101.6, 117.3)
- added REF**: Stitching_Via_0.6mm, Hella_Bauteile:Stitching_Via_0.6mm, F.Cu at (101.6, 116.1)
- added REF**: Stitching_Via_0.6mm, Hella_Bauteile:Stitching_Via_0.6mm, F.Cu at (99.1, 116.1)
- added REF**: Stitching_Via_0.6mm, Hella_Bauteile:Stitching_Via_0.6mm, F.Cu at (99.1, 118.6)
- added REF**: Stitching_Via_0.6mm, Hella_Bauteile:Stitching_Via_0.6mm, F.Cu at (101.6, 118.6)
- added T2: MUN5313DW, Package_TO_SOT_SMD:SOT-363_SC-70-6_Handsoldering, F.Cu at (87.8, 94.8)
- added T3: MUN5313DW, Package_TO_SOT_SMD:SOT-363_SC-70-6_Handsoldering, F.Cu at (100.3, 93.5)
- C51: value 390pf -> 390pF
- K1: footprint Relay_SMD:Relay_DPDT_AXICOM_IMSeries_JLeg -> Hella_Bauteile:Relay_DPDT_AXICOM_IMSeries_GullWing
- moved G*** 29.9 mm to (136.4, 124.2)
- moved C38 12.0 mm to (104.4, 112.3)
- moved R25 12.0 mm to (87.3, 120.1)
- moved R34 12.0 mm to (109.6, 118.8)
- moved R36 12.0 mm to (109.6, 121.0)
- moved C27 12.0 mm to (74.5, 113.3)
- moved C28 12.0 mm to (83.4, 122.6)
- moved C37 12.0 mm to (96.5, 112.3)
- moved C39 12.0 mm to (93.5, 119.7)
- moved Q4 12.0 mm to (89.9, 115.0)
- moved R29 12.0 mm to (88.5, 102.8)
- moved R32 12.0 mm to (112.4, 102.8)
- moved R35 12.0 mm to (90.5, 120.7)
- moved R37 12.0 mm to (100.4, 112.3)
- moved C29 12.0 mm to (81.1, 122.6)
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Connections:
- U3 pad 24: Net-(U3-Pad24) -> /EXT_INPUT_1
- U3 pad 25: Net-(U3-Pad25) -> /EXT_INPUT_2
Routing:
- net /EXT_INPUT_1: track 0.00 -> 104.0 mm, vias 0 -> 6
- net /EXT_INPUT_2: track 0.00 -> 79.4 mm, vias 0 -> 4
- net Net-(R61-Pad1): track 0.00 -> 70.0 mm, vias 0 -> 4
- net OUT_2: track 0.00 -> 61.9 mm, vias 0 -> 2
- net Net-(R63-Pad1): track 0.00 -> 58.8 mm, vias 0 -> 4
- net OUT_1: track 0.00 -> 44.7 mm, vias 0 -> 2
- net +12V: track 61.3 -> 101.0 mm, vias 0 -> 2
- net IN_2: track 0.00 -> 36.5 mm, vias 0 -> 1
- net KL31: track 812.1 -> 838.9 mm, vias 65 -> 126
- net IN_1: track 0.00 -> 18.7 mm, vias 0 -> 1
- net +12L: track 52.4 -> 68.5 mm
- net WAKE: track 39.5 -> 26.1 mm
- net Net-(C56-Pad1): track 0.00 -> 7.88 mm
- net Net-(C57-Pad1): track 0.00 -> 7.34 mm
- net Net-(Q3-Pad3): track 20.0 -> 27.2 mm
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Other:
- board size 100 x 70 mm -> 100 x 80 mm
- board text added: "Enable"
