File: Hardware/CarTablet.sch (KiCad schematic (older format))
At the start: 155 parts, among them IC1 TPS54540B-Q1, IC2 NCP81239, IC3 EZ-PD_CCG2, J1 ENABLE_KL15, J11 PD_to_USB_Hub, J12 USB_Tablet_Input, J13 USB_Hub_Output, J14 JTAG, J2 Anschluss, J4 ISP, J8 Arduino, K1 IM23GR, Q1 NTTFS4C13NTAG, Q2 NTTFS4C13NTAG, Q3 NTTFS4C13NTAG, Q4 NTTFS4C13NTAG, Q5 NTTFS4C13NTAG, Q6 FDG6335N, T1 MUN5313DW, U1 TJA1042T, U2 MCP2515-xSO, U3 ATmega328P-AU, U4 FT232RL, Y1 16 MHz, Y2 8 MHz

Commit message: V1.0 as ordered at JLCPCB
Parts:
- added C56, C57: 10nF, Capacitor_SMD:C_0805_2012Metric_Pad1.15x1.40mm_HandSolder, symbol Device:C
- added D12, D13: 100V, Diode_SMD:D_SMB_Handsoldering, symbol Device:D_TVS
- added D14, D15: 4.7V, Diode_SMD:D_SMB_Handsoldering, symbol Device:D_Schottky
- added D16, D17: BZX84B33, Package_TO_SOT_SMD:SOT-23, symbol Device:D_Zener
- added J3: I/O Expander, Hella_Bauteile:Molex_0901303208, symbol Connector_Generic:Conn_02x04_Top_Bottom
- added R55, R56, R57, R58, R61, R63: 10k, Resistor_SMD:R_0805_2012Metric_Pad1.15x1.40mm_HandSolder, symbol Device:R
- added R59, R60: 1k, Resistor_SMD:R_0805_2012Metric_Pad1.15x1.40mm_HandSolder, symbol Device:R
- added R62, R64: 150, Resistor_SMD:R_0805_2012Metric_Pad1.15x1.40mm_HandSolder, symbol Device:R
- added T2, T3: MUN5313DW, Package_TO_SOT_SMD:SOT-363_SC-70-6_Handsoldering, symbol CarTablet-rescue:MUN5313DW-Hella_Bauteile
- K1: footprint Relay_SMD:Relay_DPDT_AXICOM_IMSeries_JLeg -> Hella_Bauteile:Relay_DPDT_AXICOM_IMSeries_GullWing
Connections:
- net labels added: EXT_INPUT_1, EXT_INPUT_2, IN_1, IN_2, OUT_1, OUT_2
- wire segments 635 -> 719
Other:
- moved on the sheet: C26, D5, D6, R18, R19, R21
